Commit message: Add IMU pitch reading to urdf

File: uts_sensor_box/data_recorder/urdf/laser_scanner_description.urdf (robot description, URDF)
Before this commit: robot laser_scanner, 7 links, 6 joints
Joints:
- removed joint stabilised_to_base_link
- added joint stabilised_to_base_link_pitch: type continuous, parent base_stabilized, child base_link, origin xyz=0 0 0 rpy=0 0 0, axis 0 1 0
- added joint stabilised_to_base_link_roll: type continuous, parent base_stabilized, child base_link, origin xyz=0 0 0 rpy=0 0 0, axis 1 0 0

Commit message: Edit 2 DOF joint for IMU readings and add comments

File: uts_sensor_box/data_recorder/urdf/laser_scanner_description.urdf (robot description, URDF)
Before this commit: robot laser_scanner, 7 links, 7 joints
Links:
- added link base_pitch
- added link base_roll
Joints:
- removed joint stabilised_to_base_link_pitch
- removed joint stabilised_to_base_link_roll
- added joint scanner_orientation_pitch_to_base_link: type fixed, parent base_pitch, child base_link, origin xyz=0 0.065 0 rpy=0 0 0
- added joint scanner_orientation_roll_to_pitch: type continuous, parent base_roll, child base_pitch, origin xyz=0 0 0 rpy=0 0 0, axis 0 1 0
- added joint stabilized_to_scanner_orientation_roll: type continuous, parent base_stabilized, child base_roll, origin xyz=0 0 0 rpy=0 0 0, axis 1 0 0

Commit message: Add temporary map frame for testing

File: uts_sensor_box/data_recorder/urdf/laser_scanner_description.urdf (robot description, URDF)
Before this commit: robot laser_scanner, 9 links, 8 joints
Links:
- added link map
Joints:
- added joint map_to_footprint: type fixed, parent map, child base_footprint, origin xyz=0 0 0 rpy=0 0 0

Commit message: Change IMU TFs to fixed to test publish frequency

File: uts_sensor_box/data_recorder/urdf/laser_scanner_description.urdf (robot description, URDF)
Before this commit: robot laser_scanner, 10 links, 9 joints
Joints:
- joint scanner_orientation_roll_to_pitch: type continuous -> fixed
- joint stabilized_to_scanner_orientation_roll: type continuous -> fixed

Commit message: Remove static map frame for testing

File: uts_sensor_box/data_recorder/urdf/laser_scanner_description.urdf (robot description, URDF)
Before this commit: robot laser_scanner, 10 links, 9 joints
Links:
- removed link map
Joints:
- removed joint map_to_footprint

Commit message: Remove imu related joints and links from urdf
The urdf now only gives the TFs between the base_link and the other
parts of the robot. A dynamic publisher will eventually publish the TF
between the base_link and base_stabilized (given by the roll and pitch
values from the IMU). There will then be a static publisher publishing
the TF between the base_stabilized and the base_footprint.

File: uts_sensor_box/data_recorder/urdf/laser_scanner_description.urdf (robot description, URDF)
Before this commit: robot laser_scanner, 9 links, 8 joints
Links:
- removed link base_footprint
- removed link base_pitch
- removed link base_roll
- removed link base_stabilized
Joints:
- removed joint footprint_to_stabilised
- removed joint scanner_orientation_pitch_to_base_link
- removed joint scanner_orientation_roll_to_pitch
- removed joint stabilized_to_scanner_orientation_roll

Commit message: Fix imu orientation in urdfwq

File: uts_sensor_box/data_recorder/urdf/laser_scanner_description.urdf (robot description, URDF)
Before this commit: robot laser_scanner, 5 links, 4 joints
Joints:
- joint base_to_imu: origin xyz=-0.08 0.065 0.03 rpy=-1.57 0 0 -> xyz=-0.08 0.065 0.03 rpy=0 3.142 0

Commit message: Edit base_link to imu static transform

File: uts_sensor_box/data_recorder/urdf/laser_scanner_description.urdf (robot description, URDF)
Before this commit: robot laser_scanner, 5 links, 4 joints
Joints:
- joint base_to_imu: origin xyz=-0.08 0.065 0.03 rpy=0 3.142 0 -> xyz=-0.08 0.065 0.03 rpy=3.1415 0 0

Commit message: Remove hector_imu_to_tf pkg from launch file

File: uts_sensor_box/data_recorder/urdf/laser_scanner_description.urdf (robot description, URDF)
Before this commit: robot laser_scanner, 5 links, 4 joints
Joints:
- joint base_to_imu: origin xyz=-0.08 0.065 0.03 rpy=3.1415 0 0 -> xyz=-0.08 0.065 0.03 rpy=0 0 0

Commit message: Add imu orientation offset to URDF

File: uts_sensor_box/data_recorder/urdf/laser_scanner_description.urdf (robot description, URDF)
Before this commit: robot laser_scanner, 5 links, 4 joints
Joints:
- joint base_to_imu: origin xyz=-0.08 0.065 0.03 rpy=0 0 0 -> xyz=-0.08 0.065 0.03 rpy=3.1415 0 0

Commit message: Change orientation of imu in urdf

File: uts_sensor_box/data_recorder/urdf/laser_scanner_description.urdf (robot description, URDF)
Before this commit: robot laser_scanner, 5 links, 4 joints
Joints:
- joint base_to_imu: origin xyz=-0.08 0.065 0.03 rpy=3.1415 0 0 -> xyz=-0.08 0.065 0.03 rpy=3.1415 0 3.1415

Commit message: Change imu frame to corrected_imu frame
The imu frame is now a child of the corrected_imu frame that will be
published by the initial_tf_pub node.

File: uts_sensor_box/data_recorder/urdf/laser_scanner_description.urdf (robot description, URDF)
Before this commit: robot laser_scanner, 5 links, 4 joints
Joints:
- joint base_to_imu: child imu -> corrected_imu

Commit message: Rename imu link to corrected_imu in urdf

File: uts_sensor_box/data_recorder/urdf/laser_scanner_description.urdf (robot description, URDF)
Before this commit: robot laser_scanner, 5 links, 4 joints
Links:
- removed link imu
- added link corrected_imu

Commit message: Change imu offset in urdf to current imu

File: uts_sensor_box/data_recorder/urdf/laser_scanner_description.urdf (robot description, URDF)
Before this commit: robot laser_scanner, 5 links, 4 joints
Joints:
- joint base_to_imu: origin xyz=-0.08 0.065 0.03 rpy=3.1415 0 3.1415 -> xyz=-0.08 0.065 0.03 rpy=3.1415 0 0

Commit message: Change settings to suit new imu

File: uts_sensor_box/data_recorder/urdf/laser_scanner_description.urdf (robot description, URDF)
Before this commit: robot laser_scanner, 5 links, 4 joints
Joints:
- joint base_to_imu: origin xyz=-0.08 0.065 0.03 rpy=3.1415 0 3.1415 -> xyz=-0.08 0.065 0.03 rpy=0 3.1415 1.57

Commit message: Change base link to imu offset in urdf file
The offset is now changed to suit the new imu.

File: uts_sensor_box/data_recorder/urdf/laser_scanner_description.urdf (robot description, URDF)
Before this commit: robot laser_scanner, 5 links, 4 joints
Joints:
- joint base_to_imu: origin xyz=-0.08 0.065 0.03 rpy=3.1415 0 0 -> xyz=-0.08 0.065 0.03 rpy=0 3.1415 1.57

Commit message: Add correct transformation betwen base_link and imu

File: uts_sensor_box/data_recorder/urdf/laser_scanner_description.urdf (robot description, URDF)
Before this commit: robot laser_scanner, 5 links, 4 joints
Joints:
- joint base_to_imu: origin xyz=-0.08 0.065 0.03 rpy=0 3.1415 1.57 -> xyz=-0.08 0.065 0.03 rpy=3.1415 0 3.1415
